File: KiCAD/DSPIC33CK_Slot_Car_ESC/DSPIC33CK_Slot_Car_ESC.kicad_sch (KiCad schematic)
At the start: 0 parts

Commit message: Updated KiCAD
Parts:
- added ?: LM2623ALD, LDA14A, symbol 2022-02-26_02-50-42:LM2623ALD
- added C? (x5): 47uF, symbol Device:C_Small
- added C? (x2): C_Polarized_Small_US, symbol Device:C_Polarized_Small_US
- added C? (x2): C_Small, symbol Device:C_Small
- added D?: 20V, symbol Device:D_TVS
- added D? (x2): D_Schottky, symbol Device:D_Schottky
- added L?: L, symbol Device:L
- added Q?: Q_PMOS_DGS, symbol Device:Q_PMOS_DGS
- added R? (x5): 0R, symbol Device:R_Small_US
- added TP? (x2): 5016, digikey-footprints:Test_Point_3.43x1.78mm, symbol dk_Test-Points:5016
- added U? (x2): DSPIC33CK64MC102T, UQFN28_2N_MCH, symbol 2022-02-21_23-12-01:DSPIC33CK64MC102T
- added U?: LDK320AM30R, symbol LDK320:LDK320AM30R
Connections:
- new net: ?.5 (FREQ), C?.1, R?.1
- new net: ?.12 (SW), ?.13 (SW), C?.2, D?.2 (A), L?.2
- new net: L?.1, R?.2, R?.2
- new net: ?.10 (VDD), ?.11 (BOOT), ?.4 (EN), C?.1, D?.1 (K), R?.1, R?.2
- new net: ?.6 (FB), R?.1, R?.2
- new net +3V0: C?.1, D?.2 (A), R?.1, U?.5 (OUT)
- new net +3V3: R?.2
- new net GND: ?.2 (PGND), ?.3 (PGND), ?.9 (SGND), C?.2, C?.2, C?.2, C?.2, C?.2, C?.2, C?.2, C?.2, D?.1 (A1), Q?.2 (G), R?.1, TP?.1, U?.2 (GND)
- new net Track_Voltage: Q?.1 (D), TP?.1
- new net VBUS: C?.1, C?.1, C?.1, C?.1, C?.1, C?.1, D?.1 (K), D?.2 (A2), Q?.3 (S), U?.1 (IN), U?.3 (EN)
- no-connect marks 0 -> 5
Other:
- note added: "0-18V Input LDO is pass-through below 3V Boost converter operates with input down to 1.1V"
- note added: "3.3V Power Supply"
- note added: "Track Voltage Input"
